Commit message: add plugins

File: my_robot_description/urdf/common_propertise.xacro (robot description, xacro)
@@ -1,4 +1,4 @@
 <?xml version = "1.0"?>
-<robot xmlns:xacro="http://www.ros.org/wiki/xacro">
+<robot name="my_robot" xmlns:xacro="http://www.ros.org/wiki/xacro">
     <material name="green">
         <color rgba="0 0.6 0 1"/>

File: my_robot_description/urdf/mobile_base.xacro (robot description, xacro)
@@ -1,4 +1,5 @@
 <?xml version = "1.0"?>
-<robot xmlns:xacro="http://www.ros.org/wiki/xacro">
+<robot name="my_robot" xmlns:xacro="http://www.ros.org/wiki/xacro">
+    <xacro:include filename="$(find my_robot_description)/urdf/common_propertise.xacro" />
     <xacro:property name="base_length" value="0.6" />
     <xacro:property name="base_width" value="0.4" />
@@ -102,4 +103,29 @@
         <mu2 value="0.1" />
     </gazebo>
+    <link name="camera_link">
+        <inertial>
+            <mass value="0.20"/>
+            <inertia ixx="0.1" ixy="0.0" ixz="0.0" iyy="0.1" iyz="0.0" izz="0.1"/>
+        </inertial>
+        <visual name="visual_camera_link">
+            <geometry>
+               <mesh filename="model://Intel_RealSense_D435/meshes/realsense.dae" />
+            </geometry>
+            <material name="">
+                <color rgba="1.0 0.0 0.0 1.0"/>
+                <texture filename=""/>
+            </material>
+        </visual>
+        <collision>
+            <geometry>
+                <mesh filename="model://Intel_RealSense_D435/meshes/realsense.dae" />
+            </geometry>
+        </collision>
+    </link>
+<joint name="camera_joint" type="fixed">
+        <parent link="base_link" />
+        <child link="camera_link" />
+        <origin xyz="${base_length /3} 0 ${base_height}" rpy="0 0 0" />
+    </joint>
     <gazebo>
         <plugin filename="gz-sim-diff-drive-system" name="gz::sim::systems::DiffDrive">
@@ -132,39 +158,53 @@
     </gazebo>
     <gazebo reference="shoulder_link">
-    <sensor name="gpu_lidar" type="gpu_lidar">
-      <update_rate>10</update_rate>
-      <topic>scan</topic>
-      <gz_frame_id>shoulder_link</gz_frame_id>
-      <lidar>
-        <scan>
-          <horizontal>
-            <samples>720</samples>
-            <!--(max_angle-min_angle)/samples * resolution -->
-            <resolution>1</resolution>
-            <min_angle>-3.14156</min_angle>
-            <max_angle>3.14156</max_angle>
-          </horizontal>
-          <!-- Dirty hack for fake lidar detections with ogre 1 rendering in VM -->
-          <!-- <vertical>
+        <sensor name="gpu_lidar" type="gpu_lidar">
+            <update_rate>10</update_rate>
+            <topic>scan</topic>
+            <gz_frame_id>shoulder_link</gz_frame_id>
+            <lidar>
+                <scan>
+                    <horizontal>
+                        <samples>720</samples>
+                        <!--(max_angle-min_angle)/samples * resolution -->
+                        <resolution>1</resolution>
+                        <min_angle>-3.14156</min_angle>
+                        <max_angle>3.14156</max_angle>
+                    </horizontal>
+                    <!-- Dirty hack for fake lidar detections with ogre 1 rendering in VM -->
+                    <!-- <vertical>
               <samples>3</samples>
               <min_angle>-0.001</min_angle>
               <max_angle>0.001</max_angle>
           </vertical> -->
-        </scan>
-        <range>
-          <min>0.05</min>
-          <max>10.0</max>
-          <resolution>0.01</resolution>
-        </range>
-        <noise>
-            <type>gaussian</type>
-            <mean>0.0</mean>
-            <stddev>0.01</stddev>
-        </noise>
-        <frame_id>scan_link</frame_id>
-      </lidar>
-      <always_on>1</always_on>
-      <visualize>true</visualize>
-    </sensor>
-  </gazebo>
+                </scan>
+                <range>
+                    <min>0.05</min>
+                    <max>10.0</max>
+                    <resolution>0.01</resolution>
+                </range>
+                <noise>
+                    <type>gaussian</type>
+                    <mean>0.0</mean>
+                    <stddev>0.01</stddev>
+                </noise>
+                <frame_id>scan_link</frame_id>
+            </lidar>
+            <always_on>1</always_on>
+            <visualize>true</visualize>
+        </sensor>
+    </gazebo>
+<!-- Example for attaching a camera -->
+<gazebo reference="camera_link">
+  <sensor name="camera_sensor" type="camera">
+    <camera>
+      <horizontal_fov>1.047</horizontal_fov>
+      <image>
+        <width>640</width>
+        <height>480</height>
+      </image>
+    </camera>
+    <always_on>true</always_on>
+    <update_rate>30</update_rate>
+  </sensor>
+</gazebo>
 </robot>
